Commit message: Add floor frame and update OGV urdf

File: ogv_urdf/urdf/ogv.urdf.xacro (robot description, xacro)
@@ -14,5 +14,5 @@
       </geometry>
       <origin rpy="0 0 0" xyz="0 0 0"/>
-      <material name="black"/>
+      <material name="red"/>
     </visual>
     <collision>

File: ogv_urdf/urdf/ogv_body.urdf.xacro (robot description, xacro)
@@ -11,4 +11,7 @@
     <color rgba="1 1 1 1"/>
   </material>
+  <material name="red">
+    <color rgba="1 0 0 1"/>
+  </material>
   <link name="base_link">
   </link>
@@ -16,12 +19,12 @@
     <visual>
       <geometry>
-        <box size="0.358 0.33 0.052"/>
-      </geometry>
-      <origin rpy="0 0 0" xyz="0 0 0.026"/>
-      <material name="black"/>
-    </visual>
-    <collision>
-      <geometry>
-        <box size="0.358 0.33 0.052"/>
+        <box size="0.358 0.33 0.072"/>
+      </geometry>
+      <origin rpy="0 0 0" xyz="0 0 0.036"/>
+      <material name="black"/>
+    </visual>
+    <collision>
+      <geometry>
+        <box size="0.358 0.33 0.072"/>
       </geometry>
     </collision>
@@ -36,5 +39,5 @@
     <origin xyz="0 0 0"/>
   </joint>
-  <link name="lidar_frame">
+  <link name="base_laser">
     <visual>
       <geometry>
@@ -54,16 +57,16 @@
     </inertial>
   </link>
-  <joint name="lidar_to_base" type="fixed">
-    <parent link="base_link"/>
-    <child link="lidar_frame"/>
-    <origin xyz="0.144 0 0.114"/>
+  <joint name="laser_to_base" type="fixed">
+    <parent link="base_link"/>
+    <child link="base_laser"/>
+    <origin xyz="0.144 0 0.134"/>
   </joint>
    <link name="realsense_base_frame">
   </link>
-  <joint name="realsense_to_base" type="fixed">
-    <parent link="base_link"/>
-    <child link="realsense_base_frame"/>
-    <origin xyz="0.209 0 0.035"/>
-  </joint>
+    <joint name="realsense_to_base" type="fixed">
+      <parent link="base_link"/>
+      <child link="realsense_base_frame"/>
+      <origin xyz="0.209 0 0.02"/>
+    </joint>
 <link name="right_front_servo_holder">
     <visual>
@@ -354,4 +357,11 @@
     <origin rpy="0 0 0" xyz="0 0 -0.12"/>
   </joint>
+  <link name="floor_frame">
+  </link>
+  <joint name="floor_to_base_link_joint" type="fixed">
+    <parent link="base_link"/>
+    <child link="floor_frame"/>
+    <origin rpy="0 0 0" xyz="0 0 -0.164"/>
+  </joint>
   </xacro:macro>
 </robot>

Commit message: Standardize sensor frame names between OGV and TGV

File: ogv_urdf/urdf/ogv.urdf.xacro (robot description, xacro)
@@ -5,5 +5,5 @@
   <xacro:ogv_body >
   </xacro:ogv_body>
-  <xacro:sensor_d435 parent="realsense_base_frame">
+  <xacro:sensor_d435 parent="realsense_base_link">
     <origin xyz="0 0 0" rpy="0 0 0"/>
   </xacro:sensor_d435>
@@ -28,5 +28,5 @@
   <link name="thermal_optical_frame"/>
   <joint name="realsense_to_thermal" type="fixed">
-    <parent link="realsense_base_frame"/>
+    <parent link="realsense_base_link"/>
     <child link="thermal_frame"/>
     <origin xyz="0 0 0.033"/>

File: ogv_urdf/urdf/ogv_body.urdf.xacro (robot description, xacro)
@@ -40,5 +40,5 @@
   </joint>
   <!-- LIDAR  -->
-  <link name="base_laser">
+  <link name="base_laser_link">
     <visual>
       <geometry>
@@ -60,20 +60,20 @@
   <joint name="base_to_laser" type="fixed">
     <parent link="base_link"/>
-    <child link="base_laser"/>
+    <child link="base_laser_link"/>
     <origin xyz="0.144 0 0.134"/>
   </joint>
-  <link name="laser" />
+  <link name="laser_frame" />
   <joint name="base_laser_rotated" type="fixed">
-    <parent link="base_laser"/>
-    <child link="laser"/>
+    <parent link="base_laser_link"/>
+    <child link="laser_frame"/>
     <axis xyz="0 0 1"/>
     <origin xyz="0 0 0" rpy="0 0 3.14"/>
   </joint>
   <!-- REALSENSE CAMERA -->
-  <link name="realsense_base_frame">
+  <link name="realsense_base_link">
   </link>
   <joint name="base_to_realsense" type="fixed">
     <parent link="base_link"/>
-    <child link="realsense_base_frame"/>
+    <child link="realsense_base_link"/>
     <origin xyz="0.209 0 0.02"/>
   </joint>

Commit message: Add updated OGV UDRF for new realsense mount

File: ogv_urdf/urdf/ogv.urdf.xacro (robot description, xacro)
@@ -30,5 +30,5 @@
     <parent link="realsense_base_link"/>
     <child link="thermal_frame"/>
-    <origin xyz="0 0 0.033"/>
+    <origin xyz="0.010 0 0.040"/>
   </joint>
   <joint name="thermal_to_thermal_optical_joint" type="fixed">

File: ogv_urdf/urdf/ogv_body.urdf.xacro (robot description, xacro)
@@ -19,5 +19,5 @@
     <visual>
       <geometry>
-        <box size="0.358 0.33 0.072"/>
+        <box size="0.355 0.330 0.072"/>
       </geometry>
       <origin rpy="0 0 0" xyz="0 0 0.036"/>
@@ -26,5 +26,5 @@
     <collision>
       <geometry>
-        <box size="0.358 0.33 0.072"/>
+        <box size="0.355 0.330 0.072"/>
       </geometry>
     </collision>
@@ -76,5 +76,5 @@
     <parent link="base_link"/>
     <child link="realsense_base_link"/>
-    <origin xyz="0.209 0 0.02"/>
+    <origin xyz="0.196 0 -0.03"/>
   </joint>
   <!-- WHEELS AND SERVOS -->
